Commit message: COMMIT PLEASE

File: CAD/robot.urdf (robot description, URDF)
Before this commit: robot autonomous_drone, 6 links, 5 joints
Links:
- link ball_caster: geometry collision box size=1.8 1.8 1.41; visual box size=.5 .5 .5
- link box_body: geometry collision cylinder size=1.8 1.8 1.41; visual box size=.18 .18 .141
- link imu: geometry collision box size=1.8 1.8 1.41; visual box size=.5 .5 .5
- link lidar: geometry collision box size=1.8 1.8 1.41; visual box size=.5 .5 .5
- link wheel_left: geometry collision cylinder length=.019 radius=0.04; visual cylinder length=.019 radius=0.04
- link wheel_right: geometry collision cylinder length=.019 radius=0.04; visual cylinder length=.019 radius=0.04

Commit message: Push push push push

File: CAD/robot.urdf (robot description, URDF)
Before this commit: robot autonomous_drone, 6 links, 5 joints
Links:
- link imu: geometry collision box size=1.8 1.8 1.41; visual box size=0.021 .016 .005
- link lidar: geometry collision box size=0.0556 .0556 .0413; visual box size=0.0556 .0556 .0413

Commit message: merge everything

File: CAD/robot.urdf (robot description, URDF)
Before this commit: robot autonomous_drone, 6 links, 5 joints
Links:
- link ball_caster: geometry collision box size=1.8 1.8 1.41; visual sphere radius=.009525
Joints:
- joint left_wheel_joint: axis (none) -> 1 0 0; origin (none) -> xyz=-0.103 0.038 0.0195
- joint right_wheel_joint: axis (none) -> 1 0 0; origin (none) -> xyz=0.103 0.038 0.0195

Commit message: Fixed URDF completely.

File: CAD/robot.urdf (robot description, URDF)
Before this commit: robot autonomous_drone, 6 links, 5 joints
Links:
- link ball_caster: geometry collision sphere radius=.009525; visual sphere radius=.009525
- link box_body: geometry collision box size=.18 .18 .141; visual box size=.18 .18 .141
- link imu: geometry collision box size=0.021 .016 .005; visual box size=0.021 .016 .005
Joints:
- joint ball_joint: origin (none) -> xyz=0 -.07 -.01113
- joint imu_joint: origin (none) -> xyz=-0.0174 0.05225 0.114
- joint lidar_joint: origin (none) -> xyz=0 0 .16165

Commit message: WORKING ROBOT STATE PUBLISHER + FOXGLOVE + LIDAR RAHHHHHHHHHHHHHHHHHH

File: CAD/robot.urdf (robot description, URDF)
Before this commit: robot autonomous_drone, 6 links, 5 joints
Joints:
- joint lidar_joint: origin xyz=0 0 .16165 -> xyz=0 0 .16165 rpy=0 0 -1.5708
